Commit message: Update ur5.urdf.xacro

File: ur_description/urdf/ur5.urdf.xacro (robot description, xacro)
@@ -315,9 +315,15 @@
    <link name="camera"/>
     <joint name="$base_link_to_camera" type="fixed">
-      <parent link="${prefix}base_link"/>
+      <parent link="${prefix}base"/>
       <child link="camera"/>
       <!--origin xyz="-0.0109527 -0.7819547 1.1120832" rpy="3.1415926 0 0"/ -->
       <!--origin xyz="-0.0009527 -0.7819547 1.1120832" rpy="3.1415926 0 0"/-->
-       <origin xyz="0.0109527 -0.7819547 1.1120832" rpy="3.1415926 0 0"/>
+      <!--origin xyz="0.0259527 -0.7819547 1.1120832" rpy="3.1415926 0 0"/-->
+      <!--origin xyz="0.0182949 -1.25177516 0.3989193" rpy="-1.5707963 0 0"/-->
+      <!--origin xyz="0.0591778 -1.25177516 0.3589193" rpy="-1.5707963 0 0"/-->
+      <!--origin xyz="0.0291778 -1.20677516 0.5589193" rpy="-1.5707963 0 0"/-->
+      <origin xyz="-0.0691778 1.15077516 0.5089193" rpy="-1.5150 0.0160 -3.0716"/>
+      <!--origin xyz="-0.0491778 1.18677516 0.4589193" rpy="-1.5150 0.0160 -3.0716"/zuihou-->
+      <!--origin xyz="0.0291778 1.20677516 0.5589193" rpy="1.5707963 0 0"/-->
     </joint>
  <link name="table">
